File: hardware/liquidtile-3x3/electronics/liquidtile-3x3.sch (KiCad schematic (older format))
At the start: 15 parts

Commit message: Added pdf for Nate
Parts:
- gave numbers to parts that had none: 15
Changed lines of the file:
@@
-EESchema Schematic File Version 2
+EESchema Schematic File Version 2  date Friday, October 11, 2013 10:34:46 AM
 LIBS:power
 LIBS:device
@@
 LIBS:tlc5940nt
 LIBS:ft230x
-LIBS:arduino
-LIBS:arduino_shieldsNCL
+LIBS:liquidtile-3x3-cache
 EELAYER 27 0
 EELAYER END
@@
 $EndDescr
 $Comp
-L R R?
+L R R1
 U 1 1 5247330E
 P 6150 3350
-F 0 "R?" V 6230 3350 40  0000 C CNN
+F 0 "R1" V 6230 3350 40  0000 C CNN
 F 1 "2k" V 6157 3351 40  0000 C CNN
 F 2 "~" V 6080 3350 30  0000 C CNN
@@
 $EndComp
 $Comp
-L GND #PWR?
+L GND #PWR8
 U 1 1 5247331D
 P 6150 3750
-F 0 "#PWR?" H 6150 3750 30  0001 C CNN
+F 0 "#PWR8" H 6150 3750 30  0001 C CNN
 F 1 "GND" H 6150 3680 30  0001 C CNN
 F 2 "" H 6150 3750 60  0000 C CNN
@@
 $EndComp
 $Comp
-L GND #PWR?
+L GND #PWR13
 U 1 1 52473335
 P 7000 3750
-F 0 "#PWR?" H 7000 3750 30  0001 C CNN
+F 0 "#PWR13" H 7000 3750 30  0001 C CNN
 F 1 "GND" H 7000 3680 30  0001 C CNN
 F 2 "" H 7000 3750 60  0000 C CNN
@@
 $EndComp
 $Comp
-L GND #PWR?
+L GND #PWR6
 U 1 1 524733B6
 P 6000 1950
-F 0 "#PWR?" H 6000 1950 30  0001 C CNN
+F 0 "#PWR6" H 6000 1950 30  0001 C CNN
 F 1 "GND" H 6000 1880 30  0001 C CNN
 F 2 "" H 6000 1950 60  0000 C CNN
@@
 NoConn ~ 6300 2200
 $Comp
-L TLC5940NT U?
+L TLC5940NT U2
 U 1 1 5247369F
 P 6600 6200
-F 0 "U?" H 7350 6100 60  0000 C CNN
+F 0 "U2" H 7350 6100 60  0000 C CNN
 F 1 "TLC5940NT" V 7000 7100 60  0000 C CNN
 F 2 "~" H 6600 6200 60  0000 C CNN
@@
 $EndComp
 $Comp
-L R R?
+L R R2
 U 1 1 524736A5
 P 6150 6250
-F 0 "R?" V 6230 6250 40  0000 C CNN
+F 0 "R2" V 6230 6250 40  0000 C CNN
 F 1 "2k" V 6157 6251 40  0000 C CNN
 F 2 "~" V 6080 6250 30  0000 C CNN
@@
 $EndComp
 $Comp
-L GND #PWR?
+L GND #PWR11
 U 1 1 524736AB
 P 6150 6650
-F 0 "#PWR?" H 6150 6650 30  0001 C CNN
+F 0 "#PWR11" H 6150 6650 30  0001 C CNN
 F 1 "GND" H 6150 6580 30  0001 C CNN
 F 2 "" H 6150 6650 60  0000 C CNN
@@
 $EndComp
 $Comp
-L GND #PWR?
+L GND #PWR15
 U 1 1 524736B5
 P 7000 6650
-F 0 "#PWR?" H 7000 6650 30  0001 C CNN
+F 0 "#PWR15" H 7000 6650 30  0001 C CNN
 F 1 "GND" H 7000 6580 30  0001 C CNN
 F 2 "" H 7000 6650 60  0000 C CNN
@@
 $EndComp
 $Comp
-L GND #PWR?
+L GND #PWR9
 U 1 1 524736C2
 P 6150 4850
-F 0 "#PWR?" H 6150 4850 30  0001 C CNN
+F 0 "#PWR9" H 6150 4850 30  0001 C CNN
 F 1 "GND" H 6150 4780 30  0001 C CNN
 F 2 "" H 6150 4850 60  0000 C CNN
@@
 $EndComp
 $Comp
-L VCC #PWR?
+L VCC #PWR10
 U 1 1 524736C9
 P 6150 4950
-F 0 "#PWR?" H 6150 5050 30  0001 C CNN
+F 0 "#PWR10" H 6150 5050 30  0001 C CNN
 F 1 "VCC" H 6150 5050 30  0000 C CNN
 F 2 "" H 6150 4950 60  0000 C CNN
@@
 P4_B
 $Comp
-L TLC5940NT U?
+L TLC5940NT U1
 U 1 1 5247392D
 P 6600 3300
-F 0 "U?" H 7350 3200 60  0000 C CNN
+F 0 "U1" H 7350 3200 60  0000 C CNN
 F 1 "TLC5940NT" V 7000 4200 60  0000 C CNN
 F 2 "" H 6600 3300 60  0000 C CNN
@@
 BLANK
 $Comp
-L CONN_4 P?
+L CONN_4 P2
 U 1 1 52486604
 P 10200 1700
-F 0 "P?" V 10150 1700 50  0000 C CNN
+F 0 "P2" V 10150 1700 50  0000 C CNN
 F 1 "CONN_4" V 10250 1700 50  0000 C CNN
 F 2 "" H 10200 1700 60  0000 C CNN
@@
 $EndComp
 $Comp
-L CONN_4 P?
+L CONN_4 P3
 U 1 1 52486613
 P 10200 2300
-F 0 "P?" V 10150 2300 50  0000 C CNN
+F 0 "P3" V 10150 2300 50  0000 C CNN
 F 1 "CONN_4" V 10250 2300 50  0000 C CNN
 F 2 "" H 10200 2300 60  0000 C CNN
@@
 $EndComp
 $Comp
-L CONN_4 P?
+L CONN_4 P4
 U 1 1 52486620
 P 10200 2900
-F 0 "P?" V 10150 2900 50  0000 C CNN
+F 0 "P4" V 10150 2900 50  0000 C CNN
 F 1 "CONN_4" V 10250 2900 50  0000 C CNN
 F 2 "" H 10200 2900 60  0000 C CNN
@@
 $EndComp
 $Comp
-L CONN_4 P?
+L CONN_4 P5
 U 1 1 52486626
 P 10200 3450
-F 0 "P?" V 10150 3450 50  0000 C CNN
+F 0 "P5" V 10150 3450 50  0000 C CNN
 F 1 "CONN_4" V 10250 3450 50  0000 C CNN
 F 2 "" H 10200 3450 60  0000 C CNN
@@
 $EndComp
 $Comp
-L CONN_4 P?
+L CONN_4 P6
 U 1 1 5248662C
 P 10200 4000
-F 0 "P?" V 10150 4000 50  0000 C CNN
+F 0 "P6" V 10150 4000 50  0000 C CNN
 F 1 "CONN_4" V 10250 4000 50  0000 C CNN
 F 2 "" H 10200 4000 60  0000 C CNN
@@
 $EndComp
 $Comp
-L CONN_4 P?
+L CONN_4 P7
 U 1 1 52486632
 P 10200 4550
-F 0 "P?" V 10150 4550 50  0000 C CNN
+F 0 "P7" V 10150 4550 50  0000 C CNN
 F 1 "CONN_4" V 10250 4550 50  0000 C CNN
 F 2 "" H 10200 4550 60  0000 C CNN
@@
 $EndComp
 $Comp
-L CONN_4 P?
+L CONN_4 P8
 U 1 1 52486638
 P 10200 5100
-F 0 "P?" V 10150 5100 50  0000 C CNN
+F 0 "P8" V 10150 5100 50  0000 C CNN
 F 1 "CONN_4" V 10250 5100 50  0000 C CNN
 F 2 "" H 10200 5100 60  0000 C CNN
@@
 $EndComp
 $Comp
-L CONN_4 P?
+L CONN_4 P9
 U 1 1 5248663E
 P 10200 5650
-F 0 "P?" V 10150 5650 50  0000 C CNN
+F 0 "P9" V 10150 5650 50  0000 C CNN
 F 1 "CONN_4" V 10250 5650 50  0000 C CNN
 F 2 "" H 10200 5650 60  0000 C CNN
@@
 $EndComp
 $Comp
-L CONN_4 P?
+L CONN_4 P10
 U 1 1 52486644
 P 10200 6200
-F 0 "P?" V 10150 6200 50  0000 C CNN
+F 0 "P10" V 10150 6200 50  0000 C CNN
 F 1 "CONN_4" V 10250 6200 50  0000 C CNN
 F 2 "" H 10200 6200 60  0000 C CNN
@@
 $EndComp
 $Comp
-L +12V #PWR?
+L +12V #PWR16
 U 1 1 52486897
 P 9700 1500
-F 0 "#PWR?" H 9700 1450 20  0001 C CNN
+F 0 "#PWR16" H 9700 1450 20  0001 C CNN
 F 1 "+12V" H 9700 1600 30  0000 C CNN
 F 2 "" H 9700 1500 60  0000 C CNN
@@
 $EndComp
 $Comp
-L +12V #PWR?
+L +12V #PWR17
 U 1 1 52486915
 P 9700 2050
-F 0 "#PWR?" H 9700 2000 20  0001 C CNN
+F 0 "#PWR17" H 9700 2000 20  0001 C CNN
 F 1 "+12V" H 9700 2150 30  0000 C CNN
 F 2 "" H 9700 2050 60  0000 C CNN
@@
 $EndComp
 $Comp
-L +12V #PWR?
+L +12V #PWR18
 U 1 1 52486A08
 P 9700 2700
-F 0 "#PWR?" H 9700 2650 20  0001 C CNN
+F 0 "#PWR18" H 9700 2650 20  0001 C CNN
 F 1 "+12V" H 9700 2800 30  0000 C CNN
 F 2 "" H 9700 2700 60  0000 C CNN
@@
 $EndComp
 $Comp
-L +12V #PWR?
+L +12V #PWR19
 U 1 1 52486A10
 P 9700 3250
-F 0 "#PWR?" H 9700 3200 20  0001 C CNN
+F 0 "#PWR19" H 9700 3200 20  0001 C CNN
 F 1 "+12V" H 9700 3350 30  0000 C CNN
 F 2 "" H 9700 3250 60  0000 C CNN
@@
 $EndComp
 $Comp
-L +12V #PWR?
+L +12V #PWR20
 U 1 1 52486A18
 P 9700 3800
-F 0 "#PWR?" H 9700 3750 20  0001 C CNN
+F 0 "#PWR20" H 9700 3750 20  0001 C CNN
 F 1 "+12V" H 9700 3900 30  0000 C CNN
 F 2 "" H 9700 3800 60  0000 C CNN
@@
 $EndComp
 $Comp
-L +12V #PWR?
+L +12V #PWR21
 U 1 1 52486A20
 P 9700 4350
-F 0 "#PWR?" H 9700 4300 20  0001 C CNN
+F 0 "#PWR21" H 9700 4300 20  0001 C CNN
 F 1 "+12V" H 9700 4450 30  0000 C CNN
 F 2 "" H 9700 4350 60  0000 C CNN
@@
 $EndComp
 $Comp
-L +12V #PWR?
+L +12V #PWR22
 U 1 1 52486A28
 P 9700 4900
-F 0 "#PWR?" H 9700 4850 20  0001 C CNN
+F 0 "#PWR22" H 9700 4850 20  0001 C CNN
 F 1 "+12V" H 9700 5000 30  0000 C CNN
 F 2 "" H 9700 4900 60  0000 C CNN
@@
 $EndComp
 $Comp
-L +12V #PWR?
+L +12V #PWR23
 U 1 1 52486A30
 P 9700 5450
-F 0 "#PWR?" H 9700 5400 20  0001 C CNN
+F 0 "#PWR23" H 9700 5400 20  0001 C CNN
 F 1 "+12V" H 9700 5550 30  0000 C CNN
 F 2 "" H 9700 5450 60  0000 C CNN
@@
 $EndComp
 $Comp
-L +12V #PWR?
+L +12V #PWR24
 U 1 1 52486A38
 P 9700 6000
-F 0 "#PWR?" H 9700 5950 20  0001 C CNN
+F 0 "#PWR24" H 9700 5950 20  0001 C CNN
 F 1 "+12V" H 9700 6100 30  0000 C CNN
 F 2 "" H 9700 6000 60  0000 C CNN
@@
 $EndComp
 $Comp
-L +5V #PWR?
+L +5V #PWR12
 U 1 1 52486BC8
 P 7000 1250
-F 0 "#PWR?" H 7000 1340 20  0001 C CNN
+F 0 "#PWR12" H 7000 1340 20  0001 C CNN
 F 1 "+5V" H 7000 1340 30  0000 C CNN
 F 2 "" H 7000 1250 60  0000 C CNN
@@
 $EndComp
 $Comp
-L +5V #PWR?
+L +5V #PWR14
 U 1 1 52486BCE
 P 7000 4150
-F 0 "#PWR?" H 7000 4240 20  0001 C CNN
+F 0 "#PWR14" H 7000 4240 20  0001 C CNN
 F 1 "+5V" H 7000 4240 30  0000 C CNN
 F 2 "" H 7000 4150 60  0000 C CNN
@@
 $EndComp
 $Comp
-L +5V #PWR?
+L +5V #PWR7
 U 1 1 52486F68
 P 6000 2050
-F 0 "#PWR?" H 6000 2140 20  0001 C CNN
+F 0 "#PWR7" H 6000 2140 20  0001 C CNN
 F 1 "+5V" H 6000 2140 30  0000 C CNN
 F 2 "" H 6000 2050 60  0000 C CNN
@@
 	9550 6350 9850 6350
 $Comp
-L CONN_2 P?
+L CONN_2 P1
 U 1 1 52577969
 P 2500 2400
-F 0 "P?" V 2450 2400 40  0000 C CNN
+F 0 "P1" V 2450 2400 40  0000 C CNN
 F 1 "CONN_2" V 2550 2400 40  0000 C CNN
 F 2 "" H 2500 2400 60  0000 C CNN
@@
 $EndComp
 $Comp
-L GND #PWR?
+L GND #PWR4
 U 1 1 525779EE
 P 2950 2600
-F 0 "#PWR?" H 2950 2600 30  0001 C CNN
+F 0 "#PWR4" H 2950 2600 30  0001 C CNN
 F 1 "GND" H 2950 2530 30  0001 C CNN
 F 2 "" H 2950 2600 60  0000 C CNN
@@
 	2950 2500 2850 2500
 $Comp
-L +12V #PWR?
+L +12V #PWR3
 U 1 1 52577A68
 P 2950 2250
-F 0 "#PWR?" H 2950 2200 20  0001 C CNN
+F 0 "#PWR3" H 2950 2200 20  0001 C CNN
 F 1 "+12V" H 2950 2350 30  0000 C CNN
 F 2 "" H 2950 2250 60  0000 C CNN
@@
 NOTE: Each color of each set of 3 LEDs uses 20mA. \nEach LED section of 3 LEDs (with all 3 colors) uses\n 60mA and each pixel uses 120mA.
 $Comp
-L ARDUINO_SHIELD SHIELD?
+L ARDUINO_SHIELD SHIELD1
 U 1 1 52577B67
 P 2800 4650
-F 0 "SHIELD?" H 2450 5600 60  0000 C CNN
+F 0 "SHIELD1" H 2450 5600 60  0000 C CNN
 F 1 "ARDUINO_SHIELD" H 2850 3700 60  0000 C CNN
 F 2 "" H 2800 4650 60  0000 C CNN
@@
 Connection ~ 1550 4650
 $Comp
-L GND #PWR?
+L GND #PWR2
 U 1 1 52577C63
 P 1550 4800
-F 0 "#PWR?" H 1550 4800 30  0001 C CNN
+F 0 "#PWR2" H 1550 4800 30  0001 C CNN
 F 1 "GND" H 1550 4730 30  0001 C CNN
 F 2 "" H 1550 4800 60  0000 C CNN
@@
 $EndComp
 $Comp
-L +5V #PWR?
+L +5V #PWR1
 U 1 1 52577C72
 P 1550 4300
-F 0 "#PWR?" H 1550 4390 20  0001 C CNN
+F 0 "#PWR1" H 1550 4390 20  0001 C CNN
 F 1 "+5V" H 1550 4390 30  0000 C CNN
 F 2 "" H 1550 4300 60  0000 C CNN
@@
 NoConn ~ 3750 4550
 $Comp
-L GND #PWR?
+L GND #PWR5
 U 1 1 52577FE5
 P 4250 4050
-F 0 "#PWR?" H 4250 4050 30  0001 C CNN
+F 0 "#PWR5" H 4250 4050 30  0001 C CNN
 F 1 "GND" H 4250 3980 30  0001 C CNN
 F 2 "" H 4250 4050 60  0000 C CNN
